Commit message: Reduced gazebo robot launch instability - Fixed box to world - Pause sim on launch due to robot model not loading properly - Fixes robot shrivelling and flying around on launch

File: robot/robot_box.urdf (robot description, URDF)
Before this commit: robot simple_box, 1 links, 0 joints
Links:
- added link world
Joints:
- added joint fixed: type fixed, parent world, child box
