Commit message: Updated params for robustness - Updated torque and velocity to match MX106s

File: robot/bullet.xacro (robot description, xacro)
@@ -57,6 +57,6 @@
 	<xacro:property name="coxaupperlimit" value="2.4" />
 	<xacro:property name="coxalowerlimit" value="-2.4" />
-	<xacro:property name="coxaeffortlimit" value="6.0" />
-	<xacro:property name="coxavelocitylimit" value="3.14159265359" />
+	<xacro:property name="coxaeffortlimit" value="8.4" />
+	<xacro:property name="coxavelocitylimit" value="2.35619449" />
 	<xacro:property name="basemcoxaoffset" value ="-0.0145" />
 	<!-- coxa_t link -->
@@ -71,6 +71,6 @@
 	<xacro:property name="coxatupperlimit" value="2.4" />
 	<xacro:property name="coxatlowerlimit" value="-2.4" />
-	<xacro:property name="coxateffortlimit" value="6.0" />
-	<xacro:property name="coxatvelocitylimit" value="3.14159265359" />
+	<xacro:property name="coxateffortlimit" value="8.4" />
+	<xacro:property name="coxatvelocitylimit" value="2.35619449" />
 	<xacro:property name="coxacoxatoffset" value ="-0.02804" />
 	<xacro:property name="coxacoxatoffset2" value ="0.0457" />
@@ -87,6 +87,6 @@
 	<xacro:property name="femurupperlimit" value="2.4" />
 	<xacro:property name="femurlowerlimit" value="-2.4" />
-	<xacro:property name="femureffortlimit" value="6.0" />
-	<xacro:property name="femurvelocitylimit" value="3.141592653590" />
+	<xacro:property name="femureffortlimit" value="8.4" />
+	<xacro:property name="femurvelocitylimit" value="2.35619449" />
 	<xacro:property name="coxatfemuroffset" value="0.02898" />
 	<xacro:property name="coxatfemuroffset2" value="-0.06024" />
@@ -102,6 +102,6 @@
 	<xacro:property name="tibiaupperlimit" value="2.4" />
 	<xacro:property name="tibialowerlimit" value="-2.4" />
-	<xacro:property name="tibiaeffortlimit" value="6.0" />
-	<xacro:property name="tibiavelocitylimit" value="3.14159265359" />
+	<xacro:property name="tibiaeffortlimit" value="8.4" />
+	<xacro:property name="tibiavelocitylimit" value="2.35619449" />
 	<xacro:property name="femurtibiaoffset" value="0.114" />
 	<!-- tarsus link -->
@@ -115,6 +115,6 @@
 	<xacro:property name="tarsusupperlimit" value="2.4" />
 	<xacro:property name="tarsuslowerlimit" value="-2.4" />
-	<xacro:property name="tarsuseffortlimit" value="6.0" />
-	<xacro:property name="tarsusvelocitylimit" value="3.14159265359" />
+	<xacro:property name="tarsuseffortlimit" value="8.4" />
+	<xacro:property name="tarsusvelocitylimit" value="2.35619449" />
 	<xacro:property name="tibiatarsusoffset" value="0.114" />
 	<!-- TODO: Set individual static friction values for links instead of default 0.2 -->

Commit message: Fixed use of deprecated syntax -  Added xacro namespace - Updated colours

File: robot/bullet.xacro (robot description, xacro)
@@ -146,13 +146,13 @@
 			<origin xyz="0 0 ${BodyHeight/2}" rpy="0 0 0"/>
 			<mass value="${BodyMass}"/>
-			<box_inertia m="${BodyMass}" x="${BodyLength}" y="${BodyWidth}" z="${BodyHeight}"/>
+			<xacro:box_inertia m="${BodyMass}" x="${BodyLength}" y="${BodyWidth}" z="${BodyHeight}"/>
 		</inertial>
 	</link>
 	<!--Instantiation of legs: A:front, B:middle, C:rear-->
-	<leg prefix="AR" reflect="1" offset="1"/>
-	<leg prefix="AL" reflect="-1" offset="1"/>
-	<leg prefix="BR" reflect="1" offset="0"/>
-	<leg prefix="BL" reflect="-1" offset="0"/>
-	<leg prefix="CR" reflect="1" offset="-1" />
-	<leg prefix="CL" reflect="-1" offset="-1" />
+	<xacro:leg prefix="AR" reflect="1" offset="1"/>
+	<xacro:leg prefix="AL" reflect="-1" offset="1"/>
+	<xacro:leg prefix="BR" reflect="1" offset="0"/>
+	<xacro:leg prefix="BL" reflect="-1" offset="0"/>
+	<xacro:leg prefix="CR" reflect="1" offset="-1" />
+	<xacro:leg prefix="CL" reflect="-1" offset="-1" />
 </robot>

File: robot/macros.xacro (robot description, xacro)
@@ -6,16 +6,19 @@
 <!-- Modified by Benjamin Tam <benjamin.tam@data61.csiro.au> -->
 <!-- Modified by Samith Ashan <samith.ashan@data61.csiro.au> -->
-<robot name="weaver_boxmodel"
+<robot name="bullet_boxmodel"
     xmlns:xacro="http://www.ros.org/wiki/xacro">
-    <macro name="cylinder_inertia" params="m r h">
+    <xacro:macro name="cylinder_inertia" params="m r h">
         <inertia ixx="${m*(3*r*r+h*h)/12}" ixy = "0" ixz = "0" iyy="${m*(3*r*r+h*h)/12}" iyz = "0" izz="${m*r*r/2}" />
-    </macro>
-    <macro name="box_inertia" params="m x y z">
+    </xacro:macro>
+    <xacro:macro name="box_inertia" params="m x y z">
         <inertia ixx="${m*(y*y+z*z)/12}" ixy = "0" ixz = "0" iyy="${m*(x*x+z*z)/12}" iyz = "0" izz="${m*(x*x+z*z)/12}" />
-    </macro>
-    <macro name="sphere_inertia" params="m r">
+    </xacro:macro>
+    <xacro:macro name="sphere_inertia" params="m r">
         <inertia ixx="${2*m*r*r/5}" ixy = "0" ixz = "0" iyy="${2*m*r*r/5}" iyz = "0" izz="${2*m*r*r/5}" />
-    </macro>
-    <macro name="leg" params="prefix offset reflect">
+    </xacro:macro>
+    <material name="black">
+        <color rgba= "0 0 0 1"/>
+    </material>
+    <xacro:macro name="leg" params="prefix offset reflect">
         <!-- base_motor link (Base motor visual component is attached to the main body)-->
         <link name="${prefix}_basem_link">
@@ -37,5 +40,5 @@
             <inertial>
                 <mass value="${basemmass}"/>
-                <box_inertia m="${basemmass}" x="${basemlength}" y="${basemwidth}" z="${basemheight}"/>
+                <xacro:box_inertia m="${basemmass}" x="${basemlength}" y="${basemwidth}" z="${basemheight}"/>
             </inertial>
         </link>
@@ -53,5 +56,5 @@
                 </geometry>
                 <origin xyz="0 ${reflect*coxa_d} ${coxaheight/4}" rpy="0 0 ${reflect*coxa_pitch}"/>
-                <material name="white"/>
+                <material name="black"/>
             </visual>
             <collision>
@@ -63,5 +66,5 @@
             <inertial>
                 <mass value="${coxamass}"/>
-                <box_inertia m="${coxamass}" x="${coxalength}" y="${coxawidth}" z="${coxaheight}"/>
+                <xacro:box_inertia m="${coxamass}" x="${coxalength}" y="${coxawidth}" z="${coxaheight}"/>
             </inertial>
         </link>
@@ -92,5 +95,5 @@
                 </geometry>
                 <origin xyz="0 0 ${coxacoxatoffset}" rpy="0 0 ${coxat_yaw}"/>
-                <material name="white"/>
+                <material name="black"/>
             </visual>
             <collision>
@@ -102,5 +105,5 @@
             <inertial>
                 <mass value="${coxatmass}"/>
-                <box_inertia m="${coxatmass}" x="${coxatlength}" y="${coxatwidth}" z="${coxatheight}"/>
+                <xacro:box_inertia m="${coxatmass}" x="${coxatlength}" y="${coxatwidth}" z="${coxatheight}"/>
             </inertial>
         </link>
@@ -131,5 +134,5 @@
                 </geometry>
                 <origin xyz="0 0 0" rpy="0 0 0"/>
-                <material name="white"/>
+                <material name="black"/>
             </visual>
             <collision>
@@ -142,5 +145,5 @@
             <inertial>
                 <mass value="${femurmass}"/>
-                <box_inertia m="${femurmass}" x="${femurlength}" y="${femurwidth}" z="${femurheight}"/>
+                <xacro:box_inertia m="${femurmass}" x="${femurlength}" y="${femurwidth}" z="${femurheight}"/>
             </inertial>
         </link>
@@ -171,5 +174,5 @@
                 </geometry>
                 <origin xyz="0 0 0" rpy="0 0 0"/>
-                <material name="white"/>
+                <material name="black"/>
             </visual>
             <collision>
@@ -183,5 +186,5 @@
             <inertial>
                 <mass value="${tibiamass}"/>
-                <box_inertia m="${tibiamass}" x="${tibialength}" y="${tibiawidth}" z="${tibiaheight}"/>
+                <xacro:box_inertia m="${tibiamass}" x="${tibialength}" y="${tibiawidth}" z="${tibiaheight}"/>
             </inertial>
         </link>
@@ -212,5 +215,5 @@
                 </geometry>
                 <origin xyz="0 0 0" rpy="0 0 0"/>
-                <material name="white"/>
+                <material name="black"/>
             </visual>
             <collision>
@@ -223,5 +226,5 @@
             <inertial>
                 <mass value="${tarsusmass}"/>
-                <cylinder_inertia m="${tarsusmass}" h="${tarsuslength}" r="${tarsusradius}"/>
+                <xacro:cylinder_inertia m="${tarsusmass}" h="${tarsuslength}" r="${tarsusradius}"/>
                 <origin xyz="${tarsuslength/2} 0 0" rpy="0 -1.5708 0"/>
             </inertial>
@@ -249,5 +252,5 @@
             <mu1>${defaultmu1}</mu1>
             <mu2>${defaultmu2}</mu2>
-            <material>Gazebo/White</material>
+            <material>Gazebo/Black</material>
             <!-- <selfCollide>True</selfCollide> -->
             <gravity>True</gravity>
@@ -297,4 +300,4 @@
             <gravity>True</gravity>
         </gazebo>
-    </macro>
+    </xacro:macro>
 </robot>
